File: ContadorDePasajeros/ContadorDePasajeros.kicad_pcb (KiCad board)
At the start: 2 copper layers, 56.2 x 27.8 mm, 17 parts, among them J1 Conector_in, J3 Conector_esp, U1 ESP01

Commit message: 58% completado
Parts:
- MH1: value MountingHole -> MH1
- MH2: value MountingHole -> MH2
- MH3: value MountingHole -> MH3
- MH4: value MountingHole -> MH4
- moved C_F1 31.5 mm to (51.3, 58.5)
- moved C_F2 31.5 mm to (50.3, 64.0)
- moved Flash1 31.5 mm to (65.3, 70.5)
- moved J1 31.5 mm to (54.8, 58.5)
- moved J3 31.5 mm to (79.3, 58.5)
- moved MH1 31.5 mm to (48.5, 51.5)
- moved MH2 31.5 mm to (96.0, 51.5)
- moved MH3 31.5 mm to (48.8, 72.5)
- moved MH4 31.5 mm to (96.3, 72.5)
- moved RF_down1 31.5 mm to (69.8, 58.5)
- moved RF_up1 31.5 mm to (69.8, 65.8)
- moved R_CH1 31.5 mm to (61.2, 62.3)
- moved R_RST1 31.5 mm to (61.3, 65.8)
- moved Reset1 31.5 mm to (65.3, 54.0)
- moved Rx_down1 31.5 mm to (69.8, 62.3)
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Connections:
- net G2A renamed /Gpio2
- net TXA renamed Tx
- J1 pad 3: VCA -> +3V3
- J1 pad 4: GNA -> GND
- J3 pad 1: GNA -> GND
- J3 pad 4: CHA -> /Ch
- J3 pad 5: G0A -> /Gpio0
- J3 pad 6: RSA -> /Rs
- J3 pad 7: RXA -> /Rx_i
- J3 pad 8: VCA -> +3V3
- U1 pad 2: GNA -> GND
- U1 pad 3: CHA -> /Ch
- U1 pad 5: RSA -> /Rs
- U1 pad 6: G0A -> /Gpio0
- U1 pad 7: VCA -> +3V3
- U1 pad 8: RXA -> /Rx_i
Routing:
- net VCA: track 67.8 -> 0.50 mm, vias 1 -> 0
- net GNA: track 65.8 -> 0.04 mm, vias 1 -> 0
- net Net-(Flash1-Pad2): track 55.7 -> 0.00 mm, vias 2 -> 0
- net RSA: track 37.4 -> 0.00 mm
- net G0A: track 36.9 -> 0.00 mm
- net RXA: track 33.9 -> 0.00 mm, vias 4 -> 0
- net Tx: track 24.0 -> 0.96 mm, vias 1 -> 0
- net CHA: track 17.0 -> 0.00 mm, vias 1 -> 0
- net Rx: track 5.45 -> 0.00 mm
- net /Ch: track 0.00 -> 1.20 mm
- removed copper zone on F.Cu, net GNA
- removed copper zone on B.Cu, net VCA
Other:
- board size 56.2 x 27.8 mm -> 57 x 28 mm
- net class Default: via_dia 1 -> 1.2; via_drill 0.5 -> 0.6

Commit message: 57% completado
Parts:
- added C1: 100n, Capacitor_THT:CP_Radial_Tantal_D4.5mm_P5.00mm, F.Cu at (73.0, 37.7)
- added C2: 100u, Capacitor_THT:CP_Radial_D4.0mm_P1.50mm, F.Cu at (80.8, 39.6)
- added JP1: Jumper, Button_Switch_SMD:SW_SPST_B3U-1000P, F.Cu at (74.2, 43.2)
- added JP2: Jumper, Button_Switch_SMD:SW_SPST_B3U-1000P, F.Cu at (81.7, 35.7)
- added R1: 3k3, Resistor_SMD:R_0805_2012Metric_Pad1.15x1.40mm_HandSolder, F.Cu at (86.0, 35.0)
- added R2: 3k3, Resistor_SMD:R_0805_2012Metric_Pad1.15x1.40mm_HandSolder, F.Cu at (78.5, 42.9)
- added R3: 1k, Resistor_SMD:R_0805_2012Metric_Pad1.15x1.40mm_HandSolder, F.Cu at (86.0, 36.9)
- added R4: 2k, Resistor_SMD:R_0805_2012Metric_Pad1.15x1.40mm_HandSolder, F.Cu at (89.7, 35.0)
- added R5: 470, Resistor_SMD:R_0805_2012Metric_Pad1.15x1.40mm_HandSolder, F.Cu at (82.2, 42.9)
- added R6: 3k3, Resistor_SMD:R_0805_2012Metric_Pad1.15x1.40mm_HandSolder, F.Cu at (85.7, 38.9)

Commit message: 80% completado
Parts:
- removed C_F1: 100n, Capacitor_THT:CP_Radial_Tantal_D4.5mm_P5.00mm
- removed C_F2: 100u, Capacitor_THT:CP_Radial_D4.0mm_P1.50mm
- removed Flash1, Reset1: Jumper, Button_Switch_SMD:SW_SPST_B3U-1000P
- removed RF_down1: 470, Resistor_SMD:R_0805_2012Metric_Pad1.15x1.40mm_HandSolder
- removed RF_up1, R_CH1, R_RST1: 3k3, Resistor_SMD:R_0805_2012Metric_Pad1.15x1.40mm_HandSolder
- removed Rx_down1: 2k, Resistor_SMD:R_0805_2012Metric_Pad1.15x1.40mm_HandSolder
- removed Rx_up1: 1k, Resistor_SMD:R_0805_2012Metric_Pad1.15x1.40mm_HandSolder
- JP1, JP2, R1, R2, R3, R4, R5, R6: moved to B.Cu
- moved R1 42.6 mm to (62.5, 70.5), turned to 180 degrees
- moved R4 41.1 mm to (69.0, 70.5), turned to 180 degrees
- moved R3 34.7 mm to (62.0, 62.0)
- moved JP2 34.6 mm to (66.0, 66.5)
- moved C1 30.1 mm to (57.5, 63.5), turned to 270 degrees
- moved C2 28.9 mm to (57.0, 56.0), turned to 180 degrees
- moved R6 27.3 mm to (62.0, 52.5)
- moved R2 21.1 mm to (69.5, 62.0), turned to 180 degrees
- moved JP1 16.9 mm to (66.0, 58.0)
- moved R5 16.0 mm to (69.5, 52.5)
- moved J1 3.28 mm to (51.5, 58.5)
Routing:
- net GND: track 0.00 -> 89.7 mm, vias 0 -> 2
- net +3V3: track 0.00 -> 61.2 mm
- net /Gpio0: track 0.00 -> 44.3 mm, vias 0 -> 5
- net Tx: track 0.96 -> 32.7 mm, vias 0 -> 4
- net /Rx_i: track 0.00 -> 31.0 mm, vias 0 -> 4
- net /Rs: track 0.00 -> 20.8 mm
- net Rx: track 0.00 -> 12.4 mm, vias 0 -> 2
- net Net-(JP1-Pad2): track 0.00 -> 5.82 mm
- net /Ch: track 1.20 -> 6.60 mm
- net VCA: track 0.50 -> 0.00 mm
- removed copper zone on B.Cu, net GNA

Commit message: 88% completado
Routing:
- net /Gpio0: track 44.3 -> 45.3 mm
- added copper zone on F.Cu, net +3V3
- added copper zone on B.Cu, net GND
Other:
- board size 57 x 28 mm -> 57 x 30 mm
- board text added: "INDUSTRIA ARGENTINA"
Changed lines of the file:
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@@
   (general
     (thickness 1.6)
-    (drawings 8)
-    (tracks 138)
+    (drawings 9)
+    (tracks 144)
     (zones 0)
     (modules 17)
@@
   )
   (layers
-    (0 F.Cu power)
+    (0 F.Cu power hide)
     (31 B.Cu power hide)
     (32 B.Adhes user)
@@
     (user_trace_width 1)
     (trace_clearance 0.5)
-    (zone_clearance 0.508)
-    (zone_45_only no)
+    (zone_clearance 0.8)
+    (zone_45_only yes)
     (trace_min 0.25)
     (segment_width 0.2)
@@
     )
   )
-  (gr_text "Contador de pasajeros v1.0" (at 78.525 74.05) (layer F.SilkS)
+  (gr_text "INDUSTRIA ARGENTINA" (at 84.5 50.5) (layer F.SilkS)
     (effects (font (size 1 1) (thickness 0.25)))
   )
+  (gr_text "Contador de pasajeros v1.0" (at 78 75) (layer F.SilkS)
+    (effects (font (size 1 1) (thickness 0.25)))
+  )
   (dimension 57 (width 0.3) (layer Cmts.User)
-    (gr_text "57,000 mm" (at 72.5 82.6) (layer Cmts.User)
+    (gr_text "57,000 mm" (at 72.5 84.1) (layer Cmts.User)
       (effects (font (size 1.5 1.5) (thickness 0.3)))
     )
-    (feature1 (pts (xy 101 76) (xy 101 81.086421)))
-    (feature2 (pts (xy 44 76) (xy 44 81.086421)))
-    (crossbar (pts (xy 44 80.5) (xy 101 80.5)))
-    (arrow1a (pts (xy 101 80.5) (xy 99.873496 81.086421)))
-    (arrow1b (pts (xy 101 80.5) (xy 99.873496 79.913579)))
-    (arrow2a (pts (xy 44 80.5) (xy 45.126504 81.086421)))
-    (arrow2b (pts (xy 44 80.5) (xy 45.126504 79.913579)))
-  )
-  (dimension 28 (width 0.3) (layer Cmts.User)
-    (gr_text "28,000 mm" (at 106.6 62 270) (layer Cmts.User)
+    (feature1 (pts (xy 101 77.5) (xy 101 82.586421)))
+    (feature2 (pts (xy 44 77.5) (xy 44 82.586421)))
+    (crossbar (pts (xy 44 82) (xy 101 82)))
+    (arrow1a (pts (xy 101 82) (xy 99.873496 82.586421)))
+    (arrow1b (pts (xy 101 82) (xy 99.873496 81.413579)))
+    (arrow2a (pts (xy 44 82) (xy 45.126504 82.586421)))
+    (arrow2b (pts (xy 44 82) (xy 45.126504 81.413579)))
+  )
+  (dimension 30 (width 0.3) (layer Cmts.User)
+    (gr_text "30,000 mm" (at 106.6 62.5 270) (layer Cmts.User)
       (effects (font (size 1.5 1.5) (thickness 0.3)))
     )
-    (feature1 (pts (xy 101 76) (xy 105.086421 76)))
-    (feature2 (pts (xy 101 48) (xy 105.086421 48)))
-    (crossbar (pts (xy 104.5 48) (xy 104.5 76)))
-    (arrow1a (pts (xy 104.5 76) (xy 103.913579 74.873496)))
-    (arrow1b (pts (xy 104.5 76) (xy 105.086421 74.873496)))
-    (arrow2a (pts (xy 104.5 48) (xy 103.913579 49.126504)))
-    (arrow2b (pts (xy 104.5 48) (xy 105.086421 49.126504)))
+    (feature1 (pts (xy 101 77.5) (xy 105.086421 77.5)))
+    (feature2 (pts (xy 101 47.5) (xy 105.086421 47.5)))
+    (crossbar (pts (xy 104.5 47.5) (xy 104.5 77.5)))
+    (arrow1a (pts (xy 104.5 77.5) (xy 103.913579 76.373496)))
+    (arrow1b (pts (xy 104.5 77.5) (xy 105.086421 76.373496)))
+    (arrow2a (pts (xy 104.5 47.5) (xy 103.913579 48.626504)))
+    (arrow2b (pts (xy 104.5 47.5) (xy 105.086421 48.626504)))
   )
   (gr_text "Margen: 0.5 mm\nAncho pista: 0.5 mm\nDiametro Via: 1 mm\nTaladro via: 0.4 mm\n\nCuadricula: 0.5 mm\n\nFabricante:\nhttps://www.pcbcart.com/pcb-fab/hdi-pcb.html\n" (at 142.775 62.3) (layer Cmts.User)
     (effects (font (size 1.5 1.5) (thickness 0.3)))
   )
-  (gr_line (start 44 48) (end 101 48) (layer Edge.Cuts) (width 0.15))
-  (gr_line (start 101 76) (end 101 48.05) (layer Edge.Cuts) (width 0.15))
-  (gr_line (start 44 76) (end 44 48.05) (layer Edge.Cuts) (width 0.15))
-  (gr_line (start 101 76) (end 44 76) (layer Edge.Cuts) (width 0.15))
+  (gr_line (start 44 47.5) (end 101 47.5) (layer Edge.Cuts) (width 0.15))
+  (gr_line (start 101 77.5) (end 101 47.5) (layer Edge.Cuts) (width 0.15))
+  (gr_line (start 44 77.5) (end 44 47.5) (layer Edge.Cuts) (width 0.15))
+  (gr_line (start 101 77.5) (end 44 77.5) (layer Edge.Cuts) (width 0.15))
   (via (at 61 59.5) (size 1.2) (drill 0.6) (layers F.Cu B.Cu) (net 1))
   (segment (start 61 62) (end 61 59.5) (width 0.5) (layer B.Cu) (net 1))
@@
   (segment (start 71 73) (end 62.5 73) (width 0.5) (layer B.Cu) (net 3))
   (segment (start 62.5 73) (end 61.45 71.95) (width 0.5) (layer B.Cu) (net 3))
-  (segment (start 57.5 65) (end 59 66.5) (width 0.5) (layer B.Cu) (net 3))
   (segment (start 67 63.5) (end 68.5 62) (width 0.5) (layer B.Cu) (net 3))
-  (segment (start 62 63.5) (end 67 63.5) (width 0.5) (layer B.Cu) (net 3))
-  (segment (start 59 66.5) (end 62 63.5) (width 0.5) (layer B.Cu) (net 3))
-  (segment (start 61.45 69.05) (end 61.45 70.5) (width 0.5) (layer B.Cu) (net 3))
-  (segment (start 59 66.5) (end 61.5 69) (width 0.5) (layer B.Cu) (net 3))
-  (segment (start 61.5 69) (end 61.45 69.05) (width 0.5) (layer B.Cu) (net 3))
   (segment (start 57.42 63.58) (end 57.5 63.5) (width 0.5) (layer B.Cu) (net 3))
   (segment (start 51.5 63.58) (end 57.42 63.58) (width 0.5) (layer B.Cu) (net 3))
@@
   (segment (start 57 56) (end 57 55) (width 0.5) (layer B.Cu) (net 3))
   (segment (start 57 55) (end 59.5 52.5) (width 0.5) (layer B.Cu) (net 3))
+  (segment (start 64.5 63.5) (end 64 64) (width 0.5) (layer B.Cu) (net 3))
+  (segment (start 64.5 63.5) (end 67 63.5) (width 0.5) (layer B.Cu) (net 3))
+  (segment (start 64 64) (end 63 64) (width 0.5) (layer B.Cu) (net 3))
+  (segment (start 63 64) (end 61.5 65.5) (width 0.5) (layer B.Cu) (net 3))
+  (segment (start 57.5 65) (end 58 65.5) (width 0.5) (layer B.Cu) (net 3))
+  (segment (start 58 65.5) (end 60.5 65.5) (width 0.5) (layer B.Cu) (net 3))
+  (segment (start 61.5 65.5) (end 61 66) (width 0.5) (layer B.Cu) (net 3))
+  (segment (start 60.5 65.5) (end 61 66) (width 0.5) (layer B.Cu) (net 3))
+  (segment (start 61.45 70.5) (end 61.45 66.55) (width 0.5) (layer B.Cu) (net 3))
+  (segment (start 61.45 66.45) (end 60.5 65.5) (width 0.5) (layer B.Cu) (net 3))
+  (segment (start 61.45 66.55) (end 61.45 66.45) (width 0.5) (layer B.Cu) (net 3))
   (segment (start 67.7 70.2) (end 68 70.5) (width 0.5) (layer B.Cu) (net 4))
   (segment (start 55.12 66.12) (end 51.5 66.12) (width 0.5) (layer B.Cu) (net 4))
@@
   (segment (start 66 51.5) (end 66.5 51) (width 0.5) (layer B.Cu) (net 7))
   (segment (start 66 51.5) (end 67 50.5) (width 0.5) (layer B.Cu) (net 7))
+  (via (at 74 50.5) (size 1.2) (drill 0.6) (layers F.Cu B.Cu) (net 7))
+  (segment (start 67 50.5) (end 69.5 50.5) (width 0.5) (layer B.Cu) (net 7))
+  (segment (start 76 52.5) (end 79 52.5) (width 0.5) (layer B.Cu) (net 7))
+  (segment (start 74 50.5) (end 76 52.5) (width 0.5) (layer B.Cu) (net 7))
+  (segment (start 79 52.5) (end 82 55.5) (width 0.5) (layer B.Cu) (net 7))
+  (segment (start 82 55.5) (end 82 62.5) (width 0.5) (layer B.Cu) (net 7))
+  (segment (start 82 62.5) (end 80.87 63.63) (width 0.5) (layer B.Cu) (net 7))
+  (segment (start 80.87 63.63) (end 79.315 63.63) (width 0.5) (layer B.Cu) (net 7))
   (via (at 69.5 50.5) (size 1.2) (drill 0.6) (layers F.Cu B.Cu) (net 7))
-  (segment (start 67 50.5) (end 69.5 50.5) (width 0.5) (layer B.Cu) (net 7))
-  (via (at 74 50.5) (size 1.2) (drill 0.6) (layers F.Cu B.Cu) (net 7))
   (segment (start 69.5 50.5) (end 74 50.5) (width 0.5) (layer F.Cu) (net 7))
-  (segment (start 80.87 63.63) (end 79.315 63.63) (width 0.5) (layer B.Cu) (net 7))
-  (segment (start 82 62.5) (end 80.87 63.63) (width 0.5) (layer B.Cu) (net 7))
-  (segment (start 82 55.5) (end 82 62.5) (width 0.5) (layer B.Cu) (net 7))
-  (segment (start 79 52.5) (end 82 55.5) (width 0.5) (layer B.Cu) (net 7))
-  (segment (start 74 50.5) (end 76 52.5) (width 0.5) (layer B.Cu) (net 7))
-  (segment (start 76 52.5) (end 79 52.5) (width 0.5) (layer B.Cu) (net 7))
+  (segment (start 67 50.5) (end 68 50.5) (width 0.5) (layer B.Cu) (net 7))
   (segment (start 65.25 66.5) (end 66 65.75) (width 0.5) (layer B.Cu) (net 8))
   (segment (start 64.3 66.5) (end 65.25 66.5) (width 0.5) (layer B.Cu) (net 8))
@@
   (segment (start 67.7 53.275) (end 68.475 52.5) (width 0.5) (layer B.Cu) (net 10))
   (segment (start 67.7 54.8) (end 67.7 53.275) (width 0.5) (layer B.Cu) (net 10))
+  (zone (net 4) (net_name GND) (layer B.Cu) (hatch edge 0.508)
+    (connect_pads (clearance 0.8))
+    (min_thickness 0.5)
+    (fill yes (arc_segments 32) (thermal_gap 0.71) (thermal_bridge_width 0.71))
+    (polygon
+      (pts
+        (xy 42.5 46.5) (xy 42.5 78.5) (xy 102.5 78.5) (xy 102.5 46.5)
+      )
+    )
+  )
+  (zone (net 0) (net_name "") (layers F&B.Cu) (hatch full 0.508)
+    (connect_pads (clearance 0.8))
+    (min_thickness 0.5)
+    (keepout (tracks not_allowed) (vias not_allowed) (copperpour not_allowed))
+    (fill (arc_segments 32) (thermal_gap 0.71) (thermal_bridge_width 0.71))
+    (polygon
+      (pts
+        (xy 104.5 68.5) (xy 84.5 68.5) (xy 84.5 55.5) (xy 104.5 55.5)
+      )
+    )
+  )
+  (zone (net 3) (net_name +3V3) (layer F.Cu) (hatch edge 0.508)
+    (connect_pads (clearance 0.8))
+    (min_thickness 0.5)
+    (fill yes (arc_segments 32) (thermal_gap 0.71) (thermal_bridge_width 0.71))
+    (polygon
+      (pts
+        (xy 40.274139 80.5) (xy 40.774139 45.5) (xy 104.5 45) (xy 104 80)
+      )
+    )
+  )
+  (zone (net 0) (net_name "") (layers F&B.Cu) (hatch full 0.508)
+    (connect_pads (clearance 0.8))
+    (min_thickness 0.5)
+    (keepout (tracks not_allowed) (vias not_allowed) (copperpour not_allowed))
+    (fill (arc_segments 32) (thermal_gap 0.71) (thermal_bridge_width 0.71))
+    (polygon
+      (pts
+        (xy 92.918501 51.5) (xy 75.918501 51.5) (xy 75.918501 49.5) (xy 92.918501 49.5)
+      )
+    )
+  )
 )

Commit message: Netlist2
Parts:
- added F1: MH4, Fiducial:Fiducial_1mm_Dia_2mm_Outer, F.Cu at (73.8, 36.0)
- added F2: MH4, Fiducial:Fiducial_1mm_Dia_2mm_Outer, F.Cu at (73.8, 38.6)
- added Logo1: Logo_Open_Hardware_Small, Symbol:OSHW-Logo2_7.3x6mm_SilkScreen, F.Cu at (69.3, 37.5)

Commit message: 99% Completado
Parts:
- F2: moved to B.Cu
- moved F1 43.1 mm to (53.5, 74.0)
- moved Logo1 26.3 mm to (65.5, 63.5)
- moved F2 23.8 mm to (53.5, 51.0)
Other:
- board text added: "3v3"
- board text added: "GND"
- board text added: "Margen: 0.5 mm Ancho pista: 0.5 mm Diametro Via: 1 mm Taladro via: 0.4 mm Cuadricula: 0.5 mm Terminacion : HASL Fabricante: https://www.pcbcart.com/pcb-fab/hdi-pcb.html"
- board text added: "Rx"
- board text added: "Tx"
- board text removed: "Margen: 0.5 mm Ancho pista: 0.5 mm Diametro Via: 1 mm Taladro via: 0.4 mm Cuadricula: 0.5 mm Fabricante: https://www.pcbcart.com/pcb-fab/hdi-pcb.html"
Changed lines of the file:
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@@
   (general
     (thickness 1.6)
-    (drawings 9)
+    (drawings 13)
     (tracks 144)
     (zones 0)
@@
   )
   (layers
-    (0 F.Cu power hide)
-    (31 B.Cu power hide)
+    (0 F.Cu power)
+    (31 B.Cu power)
     (32 B.Adhes user)
     (33 F.Adhes user)
@@
     (pad_to_mask_clearance 0.2)
     (aux_axis_origin 0 0)
+    (grid_origin 53.5 74)
     (visible_elements 7FFFFFFF)
     (pcbplotparams
@@
     (tags "resistor handsolder")
     (attr smd)
-    (fp_text reference R3 (at 0 1.65) (layer B.SilkS)
+    (fp_text reference R3 (at 0 1.65 180) (layer B.SilkS)
       (effects (font (size 1 1) (thickness 0.15)) (justify mirror))
     )
@@
   )
   (module Fiducial:Fiducial_1mm_Dia_2mm_Outer (layer F.Cu)
-    (at 73.815001 36.025001)
+    (at 53.5 74)
     (descr "Circular Fiducial, 1mm bare copper top; 2mm keepout (Level A)")
     (tags marker)
     (attr virtual)
-    (fp_text reference F1 (at 0 -2) (layer F.SilkS)
-      (effects (font (size 1 1) (thickness 0.15)))
-    )
-    (fp_text value MH4 (at 0 2) (layer F.Fab)
+    (fp_text reference F1 (at -2.5 0) (layer F.SilkS) hide
+      (effects (font (size 1 1) (thickness 0.15)))
+    )
+    (fp_text value MH4 (at 0 0) (layer F.Fab)
       (effects (font (size 1 1) (thickness 0.15)))
     )
@@
       (solder_mask_margin 0.5) (clearance 0.5))
   )
-  (module Fiducial:Fiducial_1mm_Dia_2mm_Outer (layer F.Cu)
-    (at 73.815001 38.575001)
+  (module Fiducial:Fiducial_1mm_Dia_2mm_Outer (layer B.Cu)
+    (at 53.5 51)
     (descr "Circular Fiducial, 1mm bare copper top; 2mm keepout (Level A)")
     (tags marker)
     (attr virtual)
-    (fp_text reference F2 (at 0 -2) (layer F.SilkS)
-      (effects (font (size 1 1) (thickness 0.15)))
-    )
-    (fp_text value MH4 (at 0 2) (layer F.Fab)
-      (effects (font (size 1 1) (thickness 0.15)))
-    )
-    (fp_circle (center 0 0) (end 1.25 0) (layer F.CrtYd) (width 0.05))
-    (fp_text user %R (at 0 0) (layer F.Fab)
-      (effects (font (size 0.4 0.4) (thickness 0.06)))
-    )
-    (fp_circle (center 0 0) (end 1 0) (layer F.Fab) (width 0.1))
-    (pad ~ smd circle (at 0 0) (size 1 1) (layers F.Cu F.Mask)
+    (fp_text reference F2 (at 0 0) (layer B.SilkS) hide
+      (effects (font (size 1 1) (thickness 0.15)) (justify mirror))
+    )
+    (fp_text value MH4 (at 0 0) (layer B.Fab)
+      (effects (font (size 1 1) (thickness 0.15)) (justify mirror))
+    )
+    (fp_circle (center 0 0) (end 1.25 0) (layer B.CrtYd) (width 0.05))
+    (fp_text user %R (at 0 0) (layer B.Fab)
+      (effects (font (size 0.4 0.4) (thickness 0.06)) (justify mirror))
+    )
+    (fp_circle (center 0 0) (end 1 0) (layer B.Fab) (width 0.1))
+    (pad ~ smd circle (at 0 0) (size 1 1) (layers B.Cu B.Mask)
       (solder_mask_margin 0.5) (clearance 0.5))
   )
   (module Symbol:OSHW-Logo2_7.3x6mm_SilkScreen (layer F.Cu)
-    (at 69.270715 37.512715)
+    (at 65.5 63.5)
     (descr "Open Source Hardware Symbol")
     (tags "Logo Symbol OSHW")
-    (attr virtual)
+    (attr smd)
     (fp_text reference Logo1 (at 0 0) (layer F.SilkS) hide
       (effects (font (size 1 1) (thickness 0.15)))
@@
       (xy -0.113933 -2.757629) (xy -0.013056 -2.757714) (xy 0 -2.757714) (xy 0.10391 -2.757652)) (layer F.SilkS) (width 0.01))
   )
+  (gr_text GND (at 47.5 66) (layer F.SilkS)
+    (effects (font (size 1.5 1.5) (thickness 0.3)))
+  )
+  (gr_text 3v3 (at 47.5 63.5) (layer F.SilkS)
+    (effects (font (size 1.5 1.5) (thickness 0.3)))
+  )
+  (gr_text Tx (at 48 61) (layer F.SilkS)
+    (effects (font (size 1.5 1.5) (thickness 0.3)))
+  )
+  (gr_text Rx (at 48 58) (layer F.SilkS)
+    (effects (font (size 1.5 1.5) (thickness 0.3)))
+  )
   (gr_text "INDUSTRIA ARGENTINA" (at 84.5 50.5) (layer F.SilkS)
     (effects (font (size 1 1) (thickness 0.25)))
@@
     (arrow2b (pts (xy 104.5 47.5) (xy 105.086421 48.626504)))
   )
-  (gr_text "Margen: 0.5 mm\nAncho pista: 0.5 mm\nDiametro Via: 1 mm\nTaladro via: 0.4 mm\n\nCuadricula: 0.5 mm\n\nFabricante:\nhttps://www.pcbcart.com/pcb-fab/hdi-pcb.html\n" (at 142.775 62.3) (layer Cmts.User)
+  (gr_text "Margen: 0.5 mm\nAncho pista: 0.5 mm\nDiametro Via: 1 mm\nTaladro via: 0.4 mm\n\nCuadricula: 0.5 mm\nTerminacion : HASL\n\nFabricante:\nhttps://www.pcbcart.com/pcb-fab/hdi-pcb.html\n" (at 142.775 62.3) (layer Dwgs.User)
     (effects (font (size 1.5 1.5) (thickness 0.3)))
   )
