File: Contador12/Contador12.sch (KiCad schematic (older format))
At the start: 17 parts, among them J1 Conector_ESP, U2 ESP-12E

Commit message: 80% corregido
Parts:
- C1: footprint Capacitors_ThroughHole:C_Disc_D3.0mm_W1.6mm_P2.50mm -> Capacitor_THT:C_Disc_D3.0mm_W1.6mm_P2.50mm
- D1: footprint LEDs:LED_0805_HandSoldering -> LED_SMD:LED_0805_2012Metric_Pad1.15x1.40mm_HandSolder
- JP1, JP2: footprint Buttons_Switches_SMD:SW_SPST_B3U-1000P -> Button_Switch_SMD:SW_SPST_B3U-1000P
- MH1, MH2, MH3, MH4: footprint Mounting_Holes:MountingHole_2.5mm -> MountingHole:MountingHole_2.5mm
- R1, R2, R3, R4, R5, R6, R7: footprint Resistors_SMD:R_0805_HandSoldering -> Resistor_SMD:R_0805_2012Metric_Pad1.15x1.40mm_HandSolder
Changed lines of the file:
@@
 F 0 "JP1" V 7354 3777 50  0000 L CNN
 F 1 "Jumper" V 7445 3777 50  0000 L CNN
-F 2 "Buttons_Switches_SMD:SW_SPST_B3U-1000P" H 7400 3650 50  0001 C CNN
+F 2 "Button_Switch_SMD:SW_SPST_B3U-1000P" H 7400 3650 50  0001 C CNN
 F 3 "~" H 7400 3650 50  0001 C CNN
 	1    7400 3650
@@
 F 0 "JP2" V 4146 3412 50  0000 R CNN
 F 1 "Jumper" V 4055 3412 50  0000 R CNN
-F 2 "Buttons_Switches_SMD:SW_SPST_B3U-1000P" H 4100 3500 50  0001 C CNN
+F 2 "Button_Switch_SMD:SW_SPST_B3U-1000P" H 4100 3500 50  0001 C CNN
 F 3 "~" H 4100 3500 50  0001 C CNN
 	1    4100 3500
@@
 F 0 "R6" H 7470 4246 50  0000 L CNN
 F 1 "470" H 7470 4155 50  0000 L CNN
-F 2 "Resistors_SMD:R_0805_HandSoldering" V 7330 4200 50  0001 C CNN
+F 2 "Resistor_SMD:R_0805_2012Metric_Pad1.15x1.40mm_HandSolder" V 7330 4200 50  0001 C CNN
 F 3 "~" H 7400 4200 50  0001 C CNN
 	1    7400 4200
@@
 F 0 "R1" V 4750 2900 50  0000 L CNN
 F 1 "10k" V 4850 2900 50  0000 L CNN
-F 2 "Resistors_SMD:R_0805_HandSoldering" V 4580 2950 50  0001 C CNN
+F 2 "Resistor_SMD:R_0805_2012Metric_Pad1.15x1.40mm_HandSolder" V 4580 2950 50  0001 C CNN
 F 3 "~" H 4650 2950 50  0001 C CNN
 	1    4650 2950
@@
 F 0 "R2" V 4750 3100 50  0000 L CNN
 F 1 "10k" V 4850 3100 50  0000 L CNN
-F 2 "Resistors_SMD:R_0805_HandSoldering" V 4580 3150 50  0001 C CNN
+F 2 "Resistor_SMD:R_0805_2012Metric_Pad1.15x1.40mm_HandSolder" V 4580 3150 50  0001 C CNN
 F 3 "~" H 4650 3150 50  0001 C CNN
 	1    4650 3150
@@
 F 0 "R4" H 7120 2596 50  0000 L CNN
 F 1 "10k" H 7120 2505 50  0000 L CNN
-F 2 "Resistors_SMD:R_0805_HandSoldering" V 6980 2550 50  0001 C CNN
+F 2 "Resistor_SMD:R_0805_2012Metric_Pad1.15x1.40mm_HandSolder" V 6980 2550 50  0001 C CNN
 F 3 "~" H 7050 2550 50  0001 C CNN
 	1    7050 2550
@@
 F 0 "R3" H 6920 2596 50  0000 L CNN
 F 1 "10k" H 6920 2505 50  0000 L CNN
-F 2 "Resistors_SMD:R_0805_HandSoldering" V 6780 2550 50  0001 C CNN
+F 2 "Resistor_SMD:R_0805_2012Metric_Pad1.15x1.40mm_HandSolder" V 6780 2550 50  0001 C CNN
 F 3 "~" H 6850 2550 50  0001 C CNN
 	1    6850 2550
@@
 F 0 "R5" H 6920 3996 50  0000 L CNN
 F 1 "10k" H 6920 3905 50  0000 L CNN
-F 2 "Resistors_SMD:R_0805_HandSoldering" V 6780 3950 50  0001 C CNN
+F 2 "Resistor_SMD:R_0805_2012Metric_Pad1.15x1.40mm_HandSolder" V 6780 3950 50  0001 C CNN
 F 3 "~" H 6850 3950 50  0001 C CNN
 	1    6850 3950
@@
 F 0 "C1" H 4515 4046 50  0000 L CNN
 F 1 "100n" H 4515 3955 50  0000 L CNN
-F 2 "Capacitors_ThroughHole:C_Disc_D3.0mm_W1.6mm_P2.50mm" H 4438 3850 50  0001 C CNN
+F 2 "Capacitor_THT:C_Disc_D3.0mm_W1.6mm_P2.50mm" H 4438 3850 50  0001 C CNN
 F 3 "~" H 4400 4000 50  0001 C CNN
 	1    4400 4000
@@
 F 0 "R7" H 8070 3696 50  0000 L CNN
 F 1 "470" H 8070 3605 50  0000 L CNN
-F 2 "Resistors_SMD:R_0805_HandSoldering" V 7930 3650 50  0001 C CNN
+F 2 "Resistor_SMD:R_0805_2012Metric_Pad1.15x1.40mm_HandSolder" V 7930 3650 50  0001 C CNN
 F 3 "~" H 8000 3650 50  0001 C CNN
 	1    8000 3650
@@
 F 0 "D1" V 8038 4033 50  0000 R CNN
 F 1 "LED" V 7947 4033 50  0000 R CNN
-F 2 "LEDs:LED_0805_HandSoldering" H 8000 4150 50  0001 C CNN
+F 2 "LED_SMD:LED_0805_2012Metric_Pad1.15x1.40mm_HandSolder" H 8000 4150 50  0001 C CNN
 F 3 "~" H 8000 4150 50  0001 C CNN
 	1    8000 4150
@@
 F 0 "MH1" H 3750 5046 50  0000 L CNN
 F 1 "MH1" H 3750 4955 50  0000 L CNN
-F 2 "Mounting_Holes:MountingHole_2.5mm" H 3650 5000 50  0001 C CNN
+F 2 "MountingHole:MountingHole_2.5mm" H 3650 5000 50  0001 C CNN
 F 3 "~" H 3650 5000 50  0001 C CNN
 	1    3650 5000
@@
 F 0 "MH3" H 4500 5046 50  0000 L CNN
 F 1 "MH3" H 4500 4955 50  0000 L CNN
-F 2 "Mounting_Holes:MountingHole_2.5mm" H 4400 5000 50  0001 C CNN
+F 2 "MountingHole:MountingHole_2.5mm" H 4400 5000 50  0001 C CNN
 F 3 "~" H 4400 5000 50  0001 C CNN
 	1    4400 5000
@@
 F 0 "MH2" H 3750 5296 50  0000 L CNN
 F 1 "MH2" H 3750 5205 50  0000 L CNN
-F 2 "Mounting_Holes:MountingHole_2.5mm" H 3650 5250 50  0001 C CNN
+F 2 "MountingHole:MountingHole_2.5mm" H 3650 5250 50  0001 C CNN
 F 3 "~" H 3650 5250 50  0001 C CNN
 	1    3650 5250
@@
 F 0 "MH4" H 4500 5296 50  0000 L CNN
 F 1 "MH4" H 4500 5205 50  0000 L CNN
-F 2 "Mounting_Holes:MountingHole_2.5mm" H 4400 5250 50  0001 C CNN
+F 2 "MountingHole:MountingHole_2.5mm" H 4400 5250 50  0001 C CNN
 F 3 "~" H 4400 5250 50  0001 C CNN
 	1    4400 5250

Commit message: 82% completado
Parts:
- added F1, F2: MH2, Fiducial:Fiducial_1mm_Dia_2mm_Outer, symbol Mechanical:MountingHole
- added Logo1: Logo_Open_Hardware_Small, Symbol:OSHW-Symbol_13.4x12mm_SilkScreen, symbol Graphic:Logo_Open_Hardware_Small
Changed lines of the file:
@@
 Wire Wire Line
 	6850 2300 6850 2400
+$Comp
+L Mechanical:MountingHole F1
+U 1 1 5BE76892
+P 3700 5750
+F 0 "F1" H 3800 5796 50  0000 L CNN
+F 1 "MH2" H 3800 5705 50  0000 L CNN
+F 2 "Fiducial:Fiducial_1mm_Dia_2mm_Outer" H 3700 5750 50  0001 C CNN
+F 3 "~" H 3700 5750 50  0001 C CNN
+	1    3700 5750
+	1    0    0    -1
+$EndComp
+$Comp
+L Mechanical:MountingHole F2
+U 1 1 5BE76A1A
+P 3700 6100
+F 0 "F2" H 3800 6146 50  0000 L CNN
+F 1 "MH2" H 3800 6055 50  0000 L CNN
+F 2 "Fiducial:Fiducial_1mm_Dia_2mm_Outer" H 3700 6100 50  0001 C CNN
+F 3 "~" H 3700 6100 50  0001 C CNN
+	1    3700 6100
+	1    0    0    -1
+$EndComp
+$Comp
+L Graphic:Logo_Open_Hardware_Small Logo1
+U 1 1 5BE76AD4
+P 4600 5900
+F 0 "Logo1" H 4600 6175 50  0001 C CNN
+F 1 "Logo_Open_Hardware_Small" H 4600 5675 50  0001 C CNN
+F 2 "Symbol:OSHW-Symbol_13.4x12mm_SilkScreen" H 4600 5900 50  0001 C CNN
+F 3 "~" H 4600 5900 50  0001 C CNN
+	1    4600 5900
+	1    0    0    -1
+$EndComp
 $EndSCHEMATC
