File: Contador12/Contador12.kicad_pcb (KiCad board)
At the start: 2 copper layers, 43.8 x 40.5 mm, 25 parts, among them J1 Conector_ESP, U2 ESP-12E

Commit message: 80% corregido
Parts:
- removed LED: LED, LED_SMD:LED_0805_2012Metric_Pad1.15x1.40mm_HandSolder
- removed R_CH1, R_DOWN15, R_UP0, R_UP2: 10k, Resistor_SMD:R_0805_2012Metric_Pad1.15x1.40mm_HandSolder
- removed R_DOWN4, R_Program1: 470, Resistor_SMD:R_0805_2012Metric_Pad1.15x1.40mm_HandSolder
- removed Reset1: Jumper, Button_Switch_SMD:SW_SPST_B3U-1000P
- C1: footprint Capacitors_ThroughHole:C_Disc_D3.0mm_W1.6mm_P2.50mm -> Capacitor_THT:C_Disc_D3.0mm_W1.6mm_P2.50mm
- D1: footprint LEDs:LED_0805_HandSoldering -> LED_SMD:LED_0805_2012Metric_Pad1.15x1.40mm_HandSolder
- JP1, JP2: footprint Buttons_Switches_SMD:SW_SPST_B3U-1000P -> Button_Switch_SMD:SW_SPST_B3U-1000P
- MH1, MH2, MH3, MH4: footprint Mounting_Holes:MountingHole_2.5mm -> MountingHole:MountingHole_2.5mm
- R1, R2, R3, R4, R5, R6, R7: footprint Resistors_SMD:R_0805_HandSoldering -> Resistor_SMD:R_0805_2012Metric_Pad1.15x1.40mm_HandSolder
- moved R7 17.2 mm to (131.0, 84.0)
- moved R6 17.0 mm to (131.0, 99.5)
- moved R4 16.8 mm to (131.0, 88.0), turned to 0 degrees
- moved R3 16.7 mm to (131.0, 91.8)
- moved R5 16.7 mm to (131.0, 95.5)
- moved D1 14.8 mm to (126.8, 104.5), turned to 270 degrees
- moved JP1 6.83 mm to (131.1, 78.5)
- moved JP2 5.05 mm to (101.2, 92.5)
- moved R2 4.40 mm to (100.5, 86.7)
- moved R1 4.04 mm to (100.5, 82.2)
- moved C1 2.75 mm to (102.8, 98.5)
- moved MH1 2.75 mm to (100.2, 75.5)
- moved MH3 2.75 mm to (100.2, 107.0)
- moved U2 0.48 mm to (109.2, 82.8)
Routing:
- net Net-(D1-Pad2): track 0.00 -> 34.2 mm, vias 0 -> 2
- net Net-(D_4-Pad2): track 23.3 -> 0.00 mm, vias 2 -> 0
- net +3V3: track 79.9 -> 102.8 mm, vias 4 -> 2
- net /Program: track 18.0 -> 37.0 mm
- net GND: track 68.6 -> 56.1 mm, vias 2 -> 0
- net /Rx: track 40.5 -> 32.3 mm, vias 2 -> 1
- net /Reset: track 23.7 -> 17.2 mm, vias 0 -> 2
- net Net-(JP1-Pad2): track 32.7 -> 37.6 mm, vias 0 -> 2
- net Net-(R3-Pad1): track 10.8 -> 6.61 mm
- net Net-(R5-Pad1): track 10.6 -> 6.57 mm
- net Net-(R2-Pad1): track 4.75 -> 7.76 mm
- net Net-(R7-Pad1): track 10.6 -> 9.19 mm
- net /Tx: track 29.6 -> 30.9 mm
- removed copper zone on B.Cu, net +3V3
Other:
- board size 43.8 x 40.5 mm -> 46.5 x 40.5 mm

Commit message: 78% completado
Other:
- board text added: "Margen: 0.5 mm Ancho pista: 0.5 mm Diametro Via: 1 mm Taladro via: 0.4 mm Cuadricula: 0.5 mm Fabricante: https://www.pcbcart.com/pcb-fab/hdi-pcb.html"
- board text removed: "Margen: 0.5 mm Ancho pista: 0.5 mm Diametro Via: 1 mm Taladro via: 0.4 mm Cuadricula: 0.25 mm Fabricante: https://www.pcbcart.com/pcb-fab/hdi-pcb.html"
Changed lines of the file:
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@@
   (gr_line (start 142.45 111.275) (end 96 111.25) (layer Edge.Cuts) (width 0.15))
   (gr_line (start 142.475 70.75) (end 142.45 111.275) (layer Edge.Cuts) (width 0.15))
-  (gr_text "Margen: 0.5 mm\nAncho pista: 0.5 mm\nDiametro Via: 1 mm\nTaladro via: 0.4 mm\n\nCuadricula: 0.25 mm\n\nFabricante:\nhttps://www.pcbcart.com/pcb-fab/hdi-pcb.html\n" (at 182.25 91.75) (layer Cmts.User)
+  (gr_text "Margen: 0.5 mm\nAncho pista: 0.5 mm\nDiametro Via: 1 mm\nTaladro via: 0.4 mm\n\nCuadricula: 0.5 mm\n\nFabricante:\nhttps://www.pcbcart.com/pcb-fab/hdi-pcb.html\n" (at 182.25 91.75) (layer Cmts.User)
     (effects (font (size 1.5 1.5) (thickness 0.3)))
   )

Commit message: 82% completado
Parts:
- added F1: MH2, Fiducial:Fiducial_1mm_Dia_2mm_Outer, F.Cu at (169.1, 72.3)
- added F2: MH2, Fiducial:Fiducial_1mm_Dia_2mm_Outer, F.Cu at (169.1, 74.8)
- added Logo1: Logo_Open_Hardware_Small, Symbol:OSHW-Symbol_13.4x12mm_SilkScreen, F.Cu at (161.2, 77.0)

Commit message: 96% completado
Parts:
- added ?: , , F.Cu at (123.5, 112.0)
- F2, Logo1: moved to B.Cu
- moved F1 72.7 mm to (105.5, 107.5)
- moved F2 64.1 mm to (105.0, 75.5)
- moved Logo1 48.0 mm to (116.5, 94.5), turned to 180 degrees
- moved MH2 0.79 mm to (139.0, 75.0)
- moved MH1 0.56 mm to (100.5, 75.0)
- moved MH3 0.56 mm to (100.5, 106.5)
- moved MH4 0.25 mm to (139.0, 107.0)
Routing:
- added copper zone on F.Cu, net +3V3
- added copper zone on B.Cu, net GND
Other:
- board size 46.5 x 40.5 mm -> 47.5 x 41 mm
- board text added: "3v3"
- board text added: "GND"
- board text added: "IND. ARG."
- board text added: "Margen: 0.5 mm Ancho pista: 0.5 mm Diametro Via: 1 mm Taladro via: 0.4 mm Cuadricula: 0.5 mm Terminacion: HASL Fabricante: https://www.pcbcart.com/pcb-fab/hdi-pcb.html"
- board text added: "Rx"
- board text added: "Tx"
- board text removed: "Margen: 0.5 mm Ancho pista: 0.5 mm Diametro Via: 1 mm Taladro via: 0.4 mm Cuadricula: 0.5 mm Fabricante: https://www.pcbcart.com/pcb-fab/hdi-pcb.html"
